Commit message: Second commit

File: rover_description/urdf/rover.urdf (robot description, URDF)
Before this commit: robot rover, 3 links, 2 joints
Links:
- link base_link: mass 2 -> None
- link bottom_level: mass 1 -> None
- link sensor_laser: mass 1 -> None

Commit message: Lots of changes

File: rover_description/urdf/rover.urdf (robot description, URDF)
Before this commit: robot rover, 3 links, 2 joints
Links:
- added link base_footprint
- added link top_level; collision cylinder length=0.006 radius=0.11; visual cylinder length=0.006 radius=0.11
- link base_link: geometry collision box size=${base_length} ${base_width} ${base_height}; visual box size=${base_length} ${base_width} ${base_height}
Joints:
- added joint base_joint: type fixed, parent base_link, child base_footprint, origin xyz=0.0 0.0 ${-(wheel_radius+wheel_zoff)} rpy=0 0 0
- added joint joint_top_level: type fixed, parent base_link, child top_level, origin xyz=0.0 0 0.060 rpy=0 0 0

Commit message: Added articubot

File: rover_description/urdf/rover.urdf (robot description, URDF)
Before this commit: robot rover, 5 links, 4 joints
Links:
- removed link sensor_laser
Joints:
- removed joint joint_sensor_laser
